File: Red/Flash.sch (KiCad schematic (older format))
At the start: 1 part

Commit message: Made one library in the project folder with all symbols and footprints for easy sharing
Parts:
- I1: renamed from I601; symbol my_KiKAD-symbol-library:MT25QL512ABB8ESF-0SIT -> red_symbols:MT25QL512ABB8ESF-0SIT-my_KiKAD-symbol-library
Changed lines of the file:
@@
 QSPI_IO[0...3]
 $Comp
-L my_KiKAD-symbol-library:MT25QL512ABB8ESF-0SIT I601
+L red_symbols:MT25QL512ABB8ESF-0SIT-my_KiKAD-symbol-library I?
 U 1 1 5ED3CC59
 P 5650 4850
-F 0 "I601" H 5700 5425 50  0000 C CNN
+AR Path="/5ED3CC59" Ref="I?"  Part="1"
+AR Path="/5EC9A08F/5ED3CC59" Ref="I1"  Part="1"
+F 0 "I1" H 5700 5425 50  0000 C CNN
 F 1 "MT25QL512ABB8ESF-0SIT" H 5700 5334 50  0000 C CNN
 F 2 "Package_SO:SOP-16_4.55x10.3mm_P1.27mm" H 5200 5450 50  0001 C CNN

Commit message: Post design review
Parts:
- renumbered I1 to I401
Changed lines of the file:
@@
 P 5650 4850
 AR Path="/5ED3CC59" Ref="I?"  Part="1"
-AR Path="/5EC9A08F/5ED3CC59" Ref="I1"  Part="1"
-F 0 "I1" H 5700 5425 50  0000 C CNN
+AR Path="/5EC9A08F/5ED3CC59" Ref="I401"  Part="1"
+F 0 "I401" H 5700 5425 50  0000 C CNN
 F 1 "MT25QL512ABB8ESF-0SIT" H 5700 5334 50  0000 C CNN
 F 2 "Package_SO:SOP-16_4.55x10.3mm_P1.27mm" H 5200 5450 50  0001 C CNN
@@
 NoConn ~ 5000 5100
 $Comp
-L power:+3.3V #PWR0601
+L power:+3.3V #PWR0401
 U 1 1 5ED3F610
 P 6500 4400
-F 0 "#PWR0601" H 6500 4250 50  0001 C CNN
+F 0 "#PWR0401" H 6500 4250 50  0001 C CNN
 F 1 "+3.3V" H 6515 4573 50  0000 C CNN
 F 2 "" H 6500 4400 50  0001 C CNN
@@
 $EndComp
 $Comp
-L power:GND #PWR0602
+L power:GND #PWR0402
 U 1 1 5ED3FD0F
 P 6500 4700
-F 0 "#PWR0602" H 6500 4450 50  0001 C CNN
+F 0 "#PWR0402" H 6500 4450 50  0001 C CNN
 F 1 "GND" H 6505 4527 50  0000 C CNN
 F 2 "" H 6500 4700 50  0001 C CNN
