File: Red/RGBLEDs.sch (KiCad schematic (older format))
At the start: 8 parts

Commit message: updated documentation and fixed a few minor erros
Parts:
- D1: footprint my_library:LED_RGB_3.5mmx2.8mm -> Red:LED_RGB_3.5mmx2.8mm
Changed lines of the file:
@@
 F 0 "D1" H 3350 1383 50  0000 C CNN
 F 1 "LED_RGBC" H 3350 1474 50  0000 C CNN
-F 2 "my_library:LED_RGB_3.5mmx2.8mm" H 3350 1800 50  0001 C CNN
+F 2 "Red:LED_RGB_3.5mmx2.8mm" H 3350 1800 50  0001 C CNN
 F 3 "~" H 3350 1800 50  0001 C CNN
 F 4 "1497-1225-1-ND" H 3350 1850 50  0001 C CNN "digikey"

Commit message: Post design review
Parts:
- removed R302, R303, R304, R305, R306: 165, digikey-kicad-library:0603, symbol Device:R
- added R602, R603, R604, R605, R606: 270, Resistor_SMD:R_0402_1005Metric, symbol Device:R
- R601: renamed from R301; value 165 -> 270; footprint digikey-kicad-library:0603 -> Resistor_SMD:R_0402_1005Metric; digikey ERA-3AEB151V -> A129620CT-ND
- renumbered D1 to D601, D2 to D602
Connections:
- net LED1_G: now also R602.2
- net LED1_R: now also R603.2
- net LED2_B: now also R604.2
- net LED2_G: now also R605.2
- net LED2_R: now also R606.2
- net at D601.2 (GA): now also R602.1
- net at D601.1 (RA): now also R603.1
- net at D602.3 (BA): now also R604.1
- net at D602.2 (GA): now also R605.1
- net at D602.1 (RA): now also R606.1
Changed lines of the file:
@@
 $Descr A4 11693 8268
 encoding utf-8
-Sheet 7 8
+Sheet 6 8
 Title ""
 Date ""
@@
 $EndDescr
 $Comp
-L Device:LED_RGBC D1
+L Device:LED_RGBC D601
 U 1 1 5EC663E5
 P 3350 1850
-F 0 "D1" H 3350 1383 50  0000 C CNN
+F 0 "D601" H 3350 1383 50  0000 C CNN
 F 1 "LED_RGBC" H 3350 1474 50  0000 C CNN
 F 2 "Red:LED_RGB_3.5mmx2.8mm" H 3350 1800 50  0001 C CNN
@@
 $EndComp
 $Comp
-L Device:LED_RGBC D2
+L Device:LED_RGBC D602
 U 1 1 5EC6823F
 P 3350 2750
-F 0 "D2" H 3350 2283 50  0000 C CNN
+F 0 "D602" H 3350 2283 50  0000 C CNN
 F 1 "LED_RGBC" H 3350 2374 50  0000 C CNN
 F 2 "my_library:LED_RGB_3.5mmx2.8mm" H 3350 2700 50  0001 C CNN
@@
 LED2_R
 $Comp
-L power:GND #PWR0301
+L power:GND #PWR0601
 U 1 1 5EC6BECA
 P 3650 1950
-F 0 "#PWR0301" H 3650 1700 50  0001 C CNN
+F 0 "#PWR0601" H 3650 1700 50  0001 C CNN
 F 1 "GND" H 3655 1777 50  0000 C CNN
 F 2 "" H 3650 1950 50  0001 C CNN
@@
 $EndComp
 $Comp
-L power:GND #PWR0302
+L power:GND #PWR0602
 U 1 1 5EC6CC73
 P 3650 2850
-F 0 "#PWR0302" H 3650 2600 50  0001 C CNN
+F 0 "#PWR0602" H 3650 2600 50  0001 C CNN
 F 1 "GND" H 3655 2677 50  0000 C CNN
 F 2 "" H 3650 2850 50  0001 C CNN
@@
 	3650 1850 3550 1850
 $Comp
-L Device:R R301
+L Device:R R601
 U 1 1 5EC16B5D
 P 2950 1650
-F 0 "R301" V 2743 1650 50  0000 C CNN
-F 1 "165" V 2834 1650 50  0000 C CNN
-F 2 "digikey-kicad-library:0603" V 2880 1650 50  0001 C CNN
+F 0 "R601" V 2743 1650 50  0000 C CNN
+F 1 "270" V 2834 1650 50  0000 C CNN
+F 2 "Resistor_SMD:R_0402_1005Metric" V 2880 1650 50  0001 C CNN
 F 3 "~" H 2950 1650 50  0001 C CNN
-F 4 "ERA-3AEB151V" V 2950 1650 50  0001 C CNN "digikey"
+F 4 "A129620CT-ND" V 2950 1650 50  0001 C CNN "digikey"
 	1    2950 1650
-	0    1    1    0
-$EndComp
-$Comp
-L Device:R R302
-U 1 1 5EC1734E
-P 2950 1850
-F 0 "R302" V 2743 1850 50  0000 C CNN
-F 1 "165" V 2834 1850 50  0000 C CNN
-F 2 "digikey-kicad-library:0603" V 2880 1850 50  0001 C CNN
-F 3 "~" H 2950 1850 50  0001 C CNN
-F 4 "ERA-3AEB151V" V 2950 1850 50  0001 C CNN "digikey"
-	1    2950 1850
-	0    1    1    0
-$EndComp
-$Comp
-L Device:R R303
-U 1 1 5EC17627
-P 2950 2050
-F 0 "R303" V 2743 2050 50  0000 C CNN
-F 1 "165" V 2834 2050 50  0000 C CNN
-F 2 "digikey-kicad-library:0603" V 2880 2050 50  0001 C CNN
-F 3 "~" H 2950 2050 50  0001 C CNN
-F 4 "ERA-3AEB151V" V 2950 2050 50  0001 C CNN "digikey"
-	1    2950 2050
-	0    1    1    0
-$EndComp
-$Comp
-L Device:R R304
-U 1 1 5EC1785A
-P 2950 2550
-F 0 "R304" V 2743 2550 50  0000 C CNN
-F 1 "165" V 2834 2550 50  0000 C CNN
-F 2 "digikey-kicad-library:0603" V 2880 2550 50  0001 C CNN
-F 3 "~" H 2950 2550 50  0001 C CNN
-F 4 "ERA-3AEB151V" V 2950 2550 50  0001 C CNN "digikey"
-	1    2950 2550
-	0    1    1    0
-$EndComp
-$Comp
-L Device:R R305
-U 1 1 5EC17E2D
-P 2950 2750
-F 0 "R305" V 2743 2750 50  0000 C CNN
-F 1 "165" V 2834 2750 50  0000 C CNN
-F 2 "digikey-kicad-library:0603" V 2880 2750 50  0001 C CNN
-F 3 "~" H 2950 2750 50  0001 C CNN
-F 4 "ERA-3AEB151V" V 2950 2750 50  0001 C CNN "digikey"
-	1    2950 2750
-	0    1    1    0
-$EndComp
-$Comp
-L Device:R R306
-U 1 1 5EC180B2
-P 2950 2950
-F 0 "R306" V 2743 2950 50  0000 C CNN
-F 1 "165" V 2834 2950 50  0000 C CNN
-F 2 "digikey-kicad-library:0603" V 2880 2950 50  0001 C CNN
-F 3 "~" H 2950 2950 50  0001 C CNN
-F 4 "ERA-3AEB151V" V 2950 2950 50  0001 C CNN "digikey"
-	1    2950 2950
 	0    1    1    0
 $EndComp
@@
 Wire Wire Line
 	3150 1650 3100 1650
+$Comp
+L Device:R R602
+U 1 1 5ED06FFD
+P 2950 1850
+F 0 "R602" V 2743 1850 50  0000 C CNN
+F 1 "270" V 2834 1850 50  0000 C CNN
+F 2 "Resistor_SMD:R_0402_1005Metric" V 2880 1850 50  0001 C CNN
+F 3 "~" H 2950 1850 50  0001 C CNN
+F 4 "A129620CT-ND" V 2950 1850 50  0001 C CNN "digikey"
+	1    2950 1850
+	0    1    1    0
+$EndComp
+$Comp
+L Device:R R603
+U 1 1 5ED07314
+P 2950 2050
+F 0 "R603" V 2743 2050 50  0000 C CNN
+F 1 "270" V 2834 2050 50  0000 C CNN
+F 2 "Resistor_SMD:R_0402_1005Metric" V 2880 2050 50  0001 C CNN
+F 3 "~" H 2950 2050 50  0001 C CNN
+F 4 "A129620CT-ND" V 2950 2050 50  0001 C CNN "digikey"
+	1    2950 2050
+	0    1    1    0
+$EndComp
+$Comp
+L Device:R R604
+U 1 1 5ED076A1
+P 2950 2550
+F 0 "R604" V 2743 2550 50  0000 C CNN
+F 1 "270" V 2834 2550 50  0000 C CNN
+F 2 "Resistor_SMD:R_0402_1005Metric" V 2880 2550 50  0001 C CNN
+F 3 "~" H 2950 2550 50  0001 C CNN
+F 4 "A129620CT-ND" V 2950 2550 50  0001 C CNN "digikey"
+	1    2950 2550
+	0    1    1    0
+$EndComp
+$Comp
+L Device:R R605
+U 1 1 5ED07B7C
+P 2950 2750
+F 0 "R605" V 2743 2750 50  0000 C CNN
+F 1 "270" V 2834 2750 50  0000 C CNN
+F 2 "Resistor_SMD:R_0402_1005Metric" V 2880 2750 50  0001 C CNN
+F 3 "~" H 2950 2750 50  0001 C CNN
+F 4 "A129620CT-ND" V 2950 2750 50  0001 C CNN "digikey"
+	1    2950 2750
+	0    1    1    0
+$EndComp
+$Comp
+L Device:R R606
+U 1 1 5ED07E5D
+P 2950 2950
+F 0 "R606" V 2743 2950 50  0000 C CNN
+F 1 "270" V 2834 2950 50  0000 C CNN
+F 2 "Resistor_SMD:R_0402_1005Metric" V 2880 2950 50  0001 C CNN
+F 3 "~" H 2950 2950 50  0001 C CNN
+F 4 "A129620CT-ND" V 2950 2950 50  0001 C CNN "digikey"
+	1    2950 2950
+	0    1    1    0
+$EndComp
 $EndSCHEMATC

Commit message: Swapped USBC connector out for one that was available, minor Silkscreen tweaks
Parts:
- D602: footprint my_library:LED_RGB_3.5mmx2.8mm -> Red:LED_RGB_3.5mmx2.8mm
Changed lines of the file:
@@
 F 0 "D602" H 3350 2283 50  0000 C CNN
 F 1 "LED_RGBC" H 3350 2374 50  0000 C CNN
-F 2 "my_library:LED_RGB_3.5mmx2.8mm" H 3350 2700 50  0001 C CNN
+F 2 "Red:LED_RGB_3.5mmx2.8mm" H 3350 2700 50  0001 C CNN
 F 3 "~" H 3350 2700 50  0001 C CNN
 F 4 "1497-1225-1-ND" H 3350 2750 50  0001 C CNN "digikey"
