File: Red/Sensors.sch (KiCad schematic (older format))
At the start: 7 parts, among them U401 MPL115A1, U402 ICM-20948

Commit message: Post design review
Parts:
- renumbered C401 to C501, C402 to C502, C403 to C503, C404 to C504, C405 to C505, U401 to U501, U402 to U502
Changed lines of the file:
@@
 $Descr A4 11693 8268
 encoding utf-8
-Sheet 6 8
+Sheet 5 8
 Title ""
 Date ""
@@
 $EndDescr
 $Comp
-L Sensor_Motion:ICM-20948 U402
+L Sensor_Motion:ICM-20948 U502
 U 1 1 5EC1B216
 P 4600 5150
-F 0 "U402" H 4900 4400 50  0000 C CNN
+F 0 "U502" H 4900 4400 50  0000 C CNN
 F 1 "ICM-20948" H 5050 4300 50  0000 C CNN
 F 2 "Sensor_Motion:InvenSense_QFN-24_3x3mm_P0.4mm" H 4600 4150 50  0001 C CNN
@@
 $EndComp
 $Comp
-L power:GND #PWR0407
+L power:GND #PWR0507
 U 1 1 5EC1CF1F
 P 4600 6100
-F 0 "#PWR0407" H 4600 5850 50  0001 C CNN
+F 0 "#PWR0507" H 4600 5850 50  0001 C CNN
 F 1 "GND" H 4605 5927 50  0000 C CNN
 F 2 "" H 4600 6100 50  0001 C CNN
@@
 	4600 5850 4600 6100
 $Comp
-L Device:C C405
+L Device:C C505
 U 1 1 5EC1DDEF
 P 5300 5500
-F 0 "C405" H 5415 5546 50  0000 L CNN
+F 0 "C505" H 5415 5546 50  0000 L CNN
 F 1 "100nF" H 5415 5455 50  0000 L CNN
 F 2 "Capacitor_SMD:C_0201_0603Metric" H 5338 5350 50  0001 C CNN
@@
 $EndComp
 $Comp
-L Device:C C403
+L Device:C C503
 U 1 1 5EC1EB34
 P 4850 4300
-F 0 "C403" V 4598 4300 50  0000 C CNN
+F 0 "C503" V 4598 4300 50  0000 C CNN
 F 1 "100nF" V 4689 4300 50  0000 C CNN
 F 2 "Capacitor_SMD:C_0201_0603Metric" H 4888 4150 50  0001 C CNN
@@
 $EndComp
 $Comp
-L Device:C C401
+L Device:C C501
 U 1 1 5EC22D50
 P 4350 4300
-F 0 "C401" V 4098 4300 50  0000 C CNN
+F 0 "C501" V 4098 4300 50  0000 C CNN
 F 1 "100nF" V 4189 4300 50  0000 C CNN
 F 2 "Capacitor_SMD:C_0201_0603Metric" H 4388 4150 50  0001 C CNN
@@
 $EndComp
 $Comp
-L power:GND #PWR0403
+L power:GND #PWR0503
 U 1 1 5EC235D6
 P 4100 4400
-F 0 "#PWR0403" H 4100 4150 50  0001 C CNN
+F 0 "#PWR0503" H 4100 4150 50  0001 C CNN
 F 1 "GND" H 4105 4227 50  0000 C CNN
 F 2 "" H 4100 4400 50  0001 C CNN
@@
 $EndComp
 $Comp
-L power:GND #PWR0409
+L power:GND #PWR0509
 U 1 1 5EC240DE
 P 5100 4400
-F 0 "#PWR0409" H 5100 4150 50  0001 C CNN
+F 0 "#PWR0509" H 5100 4150 50  0001 C CNN
 F 1 "GND" H 5105 4227 50  0000 C CNN
 F 2 "" H 5100 4400 50  0001 C CNN
@@
 $EndComp
 $Comp
-L power:GND #PWR0411
+L power:GND #PWR0511
 U 1 1 5EC24727
 P 5300 5800
-F 0 "#PWR0411" H 5300 5550 50  0001 C CNN
+F 0 "#PWR0511" H 5300 5550 50  0001 C CNN
 F 1 "GND" H 5305 5627 50  0000 C CNN
 F 2 "" H 5300 5800 50  0001 C CNN
@@
 NoConn ~ 5100 5050
 $Comp
-L power:GND #PWR0402
+L power:GND #PWR0502
 U 1 1 5EC265FE
 P 3500 5400
-F 0 "#PWR0402" H 3500 5150 50  0001 C CNN
+F 0 "#PWR0502" H 3500 5150 50  0001 C CNN
 F 1 "GND" H 3505 5227 50  0000 C CNN
 F 2 "" H 3500 5400 50  0001 C CNN
@@
 Connection ~ 4700 4300
 $Comp
-L Sensor_Pressure:MPL115A1 U401
+L Sensor_Pressure:MPL115A1 U501
 U 1 1 5EC287DA
 P 4250 2800
-F 0 "U401" H 4794 2846 50  0000 L CNN
+F 0 "U501" H 4794 2846 50  0000 L CNN
 F 1 "MPL115A1" H 4794 2755 50  0000 L CNN
 F 2 "Package_LGA:NXP_LGA-8_3x5mm_P1.25mm_H1.2mm" H 5250 2350 50  0001 C CNN
@@
 $EndComp
 $Comp
-L Device:C C404
+L Device:C C504
 U 1 1 5EC2A160
 P 5250 2950
-F 0 "C404" H 5365 2996 50  0000 L CNN
+F 0 "C504" H 5365 2996 50  0000 L CNN
 F 1 "1uF" H 5365 2905 50  0000 L CNN
 F 2 "Capacitor_SMD:C_0402_1005Metric" H 5288 2800 50  0001 C CNN
@@
 $EndComp
 $Comp
-L power:+3.3V #PWR0404
+L power:+3.3V #PWR0504
 U 1 1 5EC2CAEF
 P 4250 1950
-F 0 "#PWR0404" H 4250 1800 50  0001 C CNN
+F 0 "#PWR0504" H 4250 1800 50  0001 C CNN
 F 1 "+3.3V" H 4265 2123 50  0000 C CNN
 F 2 "" H 4250 1950 50  0001 C CNN
@@
 $EndComp
 $Comp
-L Device:C C402
+L Device:C C502
 U 1 1 5EC2D91F
 P 4400 2050
-F 0 "C402" V 4148 2050 50  0000 C CNN
+F 0 "C502" V 4148 2050 50  0000 C CNN
 F 1 "1uF" V 4239 2050 50  0000 C CNN
 F 2 "Capacitor_SMD:C_0402_1005Metric" H 4438 1900 50  0001 C CNN
@@
 $EndComp
 $Comp
-L power:GND #PWR0408
+L power:GND #PWR0508
 U 1 1 5EC2E5F2
 P 4650 2150
-F 0 "#PWR0408" H 4650 1900 50  0001 C CNN
+F 0 "#PWR0508" H 4650 1900 50  0001 C CNN
 F 1 "GND" H 4655 1977 50  0000 C CNN
 F 2 "" H 4650 2150 50  0001 C CNN
@@
 $EndComp
 $Comp
-L power:GND #PWR0410
+L power:GND #PWR0510
 U 1 1 5EC2F1BA
 P 5250 3200
-F 0 "#PWR0410" H 5250 2950 50  0001 C CNN
+F 0 "#PWR0510" H 5250 2950 50  0001 C CNN
 F 1 "GND" H 5255 3027 50  0000 C CNN
 F 2 "" H 5250 3200 50  0001 C CNN
@@
 	4250 2050 4250 2200
 $Comp
-L power:GND #PWR0405
+L power:GND #PWR0505
 U 1 1 5EC30835
 P 4250 3400
-F 0 "#PWR0405" H 4250 3150 50  0001 C CNN
+F 0 "#PWR0505" H 4250 3150 50  0001 C CNN
 F 1 "GND" H 4255 3227 50  0000 C CNN
 F 2 "" H 4250 3400 50  0001 C CNN
@@
 $EndComp
 $Comp
-L power:+3.3V #PWR0401
+L power:+3.3V #PWR0501
 U 1 1 5EC30F0C
 P 3400 3000
-F 0 "#PWR0401" H 3400 2850 50  0001 C CNN
+F 0 "#PWR0501" H 3400 2850 50  0001 C CNN
 F 1 "+3.3V" V 3415 3128 50  0000 L CNN
 F 2 "" H 3400 3000 50  0001 C CNN
@@
 ~BARO_CS
 $Comp
-L power:+3.3V #PWR0101
+L power:+3.3V #PWR0506
 U 1 1 5EC46343
 P 4500 4000
-F 0 "#PWR0101" H 4500 3850 50  0001 C CNN
+F 0 "#PWR0506" H 4500 3850 50  0001 C CNN
 F 1 "+3.3V" H 4515 4173 50  0000 C CNN
 F 2 "" H 4500 4000 50  0001 C CNN

Commit message: Swapped USBC connector out for one that was available, minor Silkscreen tweaks
Parts:
- C501, C503, C505: digikey 490-6138-2-ND -> 490-5405-1-ND
Changed lines of the file:
@@
 F 2 "Capacitor_SMD:C_0201_0603Metric" H 5338 5350 50  0001 C CNN
 F 3 "~" H 5300 5500 50  0001 C CNN
-F 4 "490-6138-2-ND" H 5300 5500 50  0001 C CNN "digikey"
+F 4 "490-5405-1-ND" H 5300 5500 50  0001 C CNN "digikey"
 	1    5300 5500
 	1    0    0    -1
@@
 F 2 "Capacitor_SMD:C_0201_0603Metric" H 4888 4150 50  0001 C CNN
 F 3 "~" H 4850 4300 50  0001 C CNN
-F 4 "490-6138-2-ND" H 4850 4300 50  0001 C CNN "digikey"
+F 4 "490-5405-1-ND" H 4850 4300 50  0001 C CNN "digikey"
 	1    4850 4300
 	0    1    1    0
@@
 F 2 "Capacitor_SMD:C_0201_0603Metric" H 4388 4150 50  0001 C CNN
 F 3 "~" H 4350 4300 50  0001 C CNN
-F 4 "490-6138-2-ND" H 4350 4300 50  0001 C CNN "digikey"
+F 4 "490-5405-1-ND" H 4350 4300 50  0001 C CNN "digikey"
 	1    4350 4300
 	0    1    1    0
