File: Red/IOConnector.sch (KiCad schematic (older format))
At the start: 8 parts, among them J501 USB_C_Receptacle, J502 Conn_01x10, J503 Conn_01x10, U501 USBLC6-2SC6

Commit message: Made one library in the project folder with all symbols and footprints for easy sharing
Parts:
- U501: symbol Power_Protection:USBLC6-2SC6 -> red_symbols:USBLC6-2SC6-Power_Protection
Changed lines of the file:
@@
 $EndComp
 $Comp
-L Power_Protection:USBLC6-2SC6 U501
+L red_symbols:USBLC6-2SC6-Power_Protection U501
 U 1 1 5EC49DC1
 P 5550 2750
+AR Path="/5EC49DC1" Ref="U501"  Part="1"
+AR Path="/5EC43DD6/5EC49DC1" Ref="U501"  Part="1"
 F 0 "U501" V 5504 3294 50  0000 L CNN
 F 1 "USBLC6-2SC6" V 5595 3294 50  0000 L CNN

Commit message: Post design review
Parts:
- removed R503, R504: 22, Capacitor_SMD:C_0402_1005Metric, symbol Device:R
- removed U501: USBLC6-2SC6, Package_TO_SOT_SMD:SOT-23-6, symbol red_symbols:USBLC6-2SC6-Power_Protection
- added C801, C802: 27pF, Capacitor_SMD:C_0402_1005Metric, symbol Device:C
- added D801: D, Diode_SMD:D_SOD-323, symbol Device:D
- added D802: LEDY, Diode_SMD:D_0603_1608Metric_Pad1.05x0.95mm_HandSolder, symbol Device:LED
- added D803: LEDG, Diode_SMD:D_0603_1608Metric_Pad1.05x0.95mm_HandSolder, symbol Device:LED
- added R803, R804: 27, Resistor_SMD:R_0402_1005Metric, symbol Device:R
- added R805, R806, R807, R808: 10k, Resistor_SMD:R_0603_1608Metric_Pad1.05x0.95mm_HandSolder, symbol Device:R
- added R809, R810: 270, Resistor_SMD:R_0402_1005Metric, symbol Device:R
- added U801: FT230XS, Package_SO:SSOP-16_3.9x4.9mm_P0.635mm, symbol Interface_USB:FT230XS
- renumbered J501 to J801, J502 to J802, J503 to J803, R501 to R801, R502 to R802
Connections:
- net labels added: MISO, MOSI, RXD, SCLK, TXD, USBD+, USBD-, ~CTS~, ~RTS~
- net labels removed: D3, USART_RX, USART_TX, USB_D+, USB_D-
- wire segments 63 -> 82
- no-connect marks 11 -> 13

Commit message: Swapped USBC connector out for one that was available, minor Silkscreen tweaks
Parts:
- J801: footprint Connector_USB:USB_C_Receptacle_Amphenol_12401548E4-2A -> Red:USB_C_Receptacle_USB4110; digikey 12401548E4#2ACT-ND -> 2073-USB4110-GF-A-1-ND
- R805, R806, R807, R808: digikey PNM0603-50KBTR-ND -> 311-10KGRCT-ND
Changed lines of the file:
@@
 F 0 "J801" H 3607 4417 50  0000 C CNN
 F 1 "USB_C_Receptacle" H 3607 4326 50  0000 C CNN
-F 2 "Connector_USB:USB_C_Receptacle_Amphenol_12401548E4-2A" H 3650 3150 50  0001 C CNN
+F 2 "Red:USB_C_Receptacle_USB4110" H 3650 3150 50  0001 C CNN
 F 3 "https://www.usb.org/sites/default/files/documents/usb_type-c.zip" H 3650 3150 50  0001 C CNN
-F 4 "12401548E4#2ACT-ND" H 3500 3150 50  0001 C CNN "digikey"
+F 4 "2073-USB4110-GF-A-1-ND" H 3500 3150 50  0001 C CNN "digikey"
 	1    3500 3150
 	1    0    0    -1
@@
 F 2 "Resistor_SMD:R_0603_1608Metric_Pad1.05x0.95mm_HandSolder" V 7530 950 50  0001 C CNN
 F 3 "~" H 7600 950 50  0001 C CNN
-F 4 "PNM0603-50KBTR-ND" H 7600 950 50  0001 C CNN "digikey"
+F 4 "311-10KGRCT-ND" H 7600 950 50  0001 C CNN "digikey"
 	1    7600 950
 	0    -1   -1   0
@@
 F 2 "Resistor_SMD:R_0603_1608Metric_Pad1.05x0.95mm_HandSolder" V 7530 1200 50  0001 C CNN
 F 3 "~" H 7600 1200 50  0001 C CNN
-F 4 "PNM0603-50KBTR-ND" H 7600 1200 50  0001 C CNN "digikey"
+F 4 "311-10KGRCT-ND" H 7600 1200 50  0001 C CNN "digikey"
 	1    7600 1200
 	0    -1   -1   0
@@
 F 2 "Resistor_SMD:R_0603_1608Metric_Pad1.05x0.95mm_HandSolder" V 7530 1450 50  0001 C CNN
 F 3 "~" H 7600 1450 50  0001 C CNN
-F 4 "PNM0603-50KBTR-ND" H 7600 1450 50  0001 C CNN "digikey"
+F 4 "311-10KGRCT-ND" H 7600 1450 50  0001 C CNN "digikey"
 	1    7600 1450
 	0    -1   -1   0
@@
 F 2 "Resistor_SMD:R_0603_1608Metric_Pad1.05x0.95mm_HandSolder" V 7530 1700 50  0001 C CNN
 F 3 "~" H 7600 1700 50  0001 C CNN
-F 4 "PNM0603-50KBTR-ND" H 7600 1700 50  0001 C CNN "digikey"
+F 4 "311-10KGRCT-ND" H 7600 1700 50  0001 C CNN "digikey"
 	1    7600 1700
 	0    -1   -1   0

Commit message: Created schematic changes for Red V1.1
Parts:
- added D?: D_Schottky, symbol Device:D_Schottky
Connections:
- wire segments 82 -> 86
Changed lines of the file:
@@
 Wire Wire Line
 	5450 2000 5450 2050
+$Comp
+L Device:D_Schottky D?
+U 1 1 5EEE9A9A
+P 4850 1700
+F 0 "D?" H 4850 1483 50  0000 C CNN
+F 1 "D_Schottky" H 4850 1574 50  0000 C CNN
+F 2 "" H 4850 1700 50  0001 C CNN
+F 3 "~" H 4850 1700 50  0001 C CNN
+	1    4850 1700
+	-1   0    0    1
+$EndComp
+$Comp
+L power:+5V #PWR?
+U 1 1 5EEEAC0A
+P 5150 1550
+F 0 "#PWR?" H 5150 1400 50  0001 C CNN
+F 1 "+5V" H 5165 1723 50  0000 C CNN
+F 2 "" H 5150 1550 50  0001 C CNN
+F 3 "" H 5150 1550 50  0001 C CNN
+	1    5150 1550
+	1    0    0    -1
+$EndComp
+$Comp
+L power:VBUS #PWR?
+U 1 1 5EEEB1B1
+P 4600 1550
+F 0 "#PWR?" H 4600 1400 50  0001 C CNN
+F 1 "VBUS" H 4615 1723 50  0000 C CNN
+F 2 "" H 4600 1550 50  0001 C CNN
+F 3 "" H 4600 1550 50  0001 C CNN
+	1    4600 1550
+	1    0    0    -1
+$EndComp
+Wire Wire Line
+	4600 1550 4600 1700
+Wire Wire Line
+	4600 1700 4700 1700
+Wire Wire Line
+	5000 1700 5150 1700
+Wire Wire Line
+	5150 1700 5150 1550
 $EndSCHEMATC

Commit message: Added footprint for diode and reannoted schematics
Parts:
- D801: renamed from D?; footprint (none) -> Diode_SMD:D_SOD-323_HandSoldering; digikey (none) -> BAT54HT1GOSCT-ND
- renumbered D801 to D802, D802 to D803, D803 to D804
Changed lines of the file:
@@
 $EndComp
 $Comp
-L power:GND #PWR0804
+L power:GND #PWR0805
 U 1 1 5EC6BC44
 P 4850 2450
-F 0 "#PWR0804" H 4850 2200 50  0001 C CNN
+F 0 "#PWR0805" H 4850 2200 50  0001 C CNN
 F 1 "GND" H 4850 2300 50  0000 C CNN
 F 2 "" H 4850 2450 50  0001 C CNN
@@
 NoConn ~ 3200 4750
 $Comp
-L power:GND #PWR0808
+L power:GND #PWR0810
 U 1 1 5EC79ACA
 P 5900 6350
-F 0 "#PWR0808" H 5900 6100 50  0001 C CNN
+F 0 "#PWR0810" H 5900 6100 50  0001 C CNN
 F 1 "GND" H 5905 6177 50  0000 C CNN
 F 2 "" H 5900 6350 50  0001 C CNN
@@
 	5900 6050 5900 6150
 $Comp
-L power:+3.3V #PWR0807
+L power:+3.3V #PWR0809
 U 1 1 5EC7D416
 P 5900 5250
-F 0 "#PWR0807" H 5900 5100 50  0001 C CNN
+F 0 "#PWR0809" H 5900 5100 50  0001 C CNN
 F 1 "+3.3V" H 5915 5423 50  0000 C CNN
 F 2 "" H 5900 5250 50  0001 C CNN
@@
 $EndComp
 $Comp
-L power:+5V #PWR0809
+L power:+5V #PWR0811
 U 1 1 5EC7F1B0
 P 6000 5550
-F 0 "#PWR0809" H 6000 5400 50  0001 C CNN
+F 0 "#PWR0811" H 6000 5400 50  0001 C CNN
 F 1 "+5V" H 6015 5723 50  0000 C CNN
 F 2 "" H 6000 5550 50  0001 C CNN
@@
 D2
 $Comp
-L power:GND #PWR0811
+L power:GND #PWR0813
 U 1 1 5EC9144C
 P 6100 5050
-F 0 "#PWR0811" H 6100 4800 50  0001 C CNN
+F 0 "#PWR0813" H 6100 4800 50  0001 C CNN
 F 1 "GND" H 6105 4877 50  0000 C CNN
 F 2 "" H 6100 5050 50  0001 C CNN
@@
 $EndComp
 $Comp
-L power:GND #PWR0813
+L power:GND #PWR0815
 U 1 1 5ECB38AB
 P 6300 3650
-F 0 "#PWR0813" H 6300 3400 50  0001 C CNN
+F 0 "#PWR0815" H 6300 3400 50  0001 C CNN
 F 1 "GND" H 6305 3477 50  0000 C CNN
 F 2 "" H 6300 3650 50  0001 C CNN
@@
 $EndComp
 $Comp
-L power:VBUS #PWR0810
+L power:VBUS #PWR0812
 U 1 1 5ECC244A
 P 6100 2050
-F 0 "#PWR0810" H 6100 1900 50  0001 C CNN
+F 0 "#PWR0812" H 6100 1900 50  0001 C CNN
 F 1 "VBUS" H 6115 2223 50  0000 C CNN
 F 2 "" H 6100 2050 50  0001 C CNN
@@
 	6100 2050 6100 2150
 $Comp
-L power:+3.3V #PWR0812
+L power:+3.3V #PWR0814
 U 1 1 5ECC36DA
 P 6300 2050
-F 0 "#PWR0812" H 6300 1900 50  0001 C CNN
+F 0 "#PWR0814" H 6300 1900 50  0001 C CNN
 F 1 "+3.3V" H 6315 2223 50  0000 C CNN
 F 2 "" H 6300 2050 50  0001 C CNN
@@
 Connection ~ 4100 2850
 $Comp
-L power:+3.3V #PWR0805
+L power:+3.3V #PWR0807
 U 1 1 5ECCB156
 P 5400 3050
-F 0 "#PWR0805" H 5400 2900 50  0001 C CNN
+F 0 "#PWR0807" H 5400 2900 50  0001 C CNN
 F 1 "+3.3V" V 5300 3050 50  0000 L CNN
 F 2 "" H 5400 3050 50  0001 C CNN
@@
 	5400 3050 5500 3050
 $Comp
-L power:+3.3V #PWR0806
+L power:+3.3V #PWR0808
 U 1 1 5ECCE6FD
 P 5450 2000
-F 0 "#PWR0806" H 5450 1850 50  0001 C CNN
+F 0 "#PWR0808" H 5450 1850 50  0001 C CNN
 F 1 "+3.3V" H 5465 2173 50  0000 C CNN
 F 2 "" H 5450 2000 50  0001 C CNN
@@
 Connection ~ 4550 3550
 $Comp
-L power:+3.3V #PWR0815
+L power:+3.3V #PWR0816
 U 1 1 5ECE38AE
 P 7350 850
-F 0 "#PWR0815" H 7350 700 50  0001 C CNN
+F 0 "#PWR0816" H 7350 700 50  0001 C CNN
 F 1 "+3.3V" H 7365 1023 50  0000 C CNN
 F 2 "" H 7350 850 50  0001 C CNN
@@
 $EndComp
 $Comp
-L Device:LED D802
+L Device:LED D803
 U 1 1 5ED16EA5
 P 7600 2900
-F 0 "D802" V 7650 3100 50  0000 R CNN
+F 0 "D803" V 7650 3100 50  0000 R CNN
 F 1 "LEDY" V 7550 3100 50  0000 R CNN
 F 2 "Diode_SMD:D_0603_1608Metric_Pad1.05x0.95mm_HandSolder" H 7600 2900 50  0001 C CNN
@@
 $EndComp
 $Comp
-L Device:LED D803
+L Device:LED D804
 U 1 1 5ED17DD2
 P 7750 2800
-F 0 "D803" V 7789 2683 50  0000 R CNN
+F 0 "D804" V 7789 2683 50  0000 R CNN
 F 1 "LEDG" V 7698 2683 50  0000 R CNN
 F 2 "Diode_SMD:D_0603_1608Metric_Pad1.05x0.95mm_HandSolder" H 7750 2800 50  0001 C CNN
@@
 	7600 2750 7600 2650
 $Comp
-L power:+3.3V #PWR0816
+L power:+3.3V #PWR0817
 U 1 1 5ED3F752
 P 7600 2200
-F 0 "#PWR0816" H 7600 2050 50  0001 C CNN
+F 0 "#PWR0817" H 7600 2050 50  0001 C CNN
 F 1 "+3.3V" H 7615 2373 50  0000 C CNN
 F 2 "" H 7600 2200 50  0001 C CNN
@@
 MISO
 $Comp
-L Device:D D801
+L Device:D D802
 U 1 1 5EDA1953
 P 5450 2200
-F 0 "D801" V 5404 2279 50  0000 L CNN
+F 0 "D802" V 5404 2279 50  0000 L CNN
 F 1 "D" V 5495 2279 50  0000 L CNN
 F 2 "Diode_SMD:D_SOD-323" H 5450 2200 50  0001 C CNN
@@
 	5450 2000 5450 2050
 $Comp
-L Device:D_Schottky D?
+L Device:D_Schottky D801
 U 1 1 5EEE9A9A
 P 4850 1700
-F 0 "D?" H 4850 1483 50  0000 C CNN
+F 0 "D801" H 4850 1483 50  0000 C CNN
 F 1 "D_Schottky" H 4850 1574 50  0000 C CNN
-F 2 "" H 4850 1700 50  0001 C CNN
+F 2 "Diode_SMD:D_SOD-323_HandSoldering" H 4850 1700 50  0001 C CNN
 F 3 "~" H 4850 1700 50  0001 C CNN
+F 4 "BAT54HT1GOSCT-ND" H 4850 1700 50  0001 C CNN "digikey"
 	1    4850 1700
 	-1   0    0    1
 $EndComp
 $Comp
-L power:+5V #PWR?
+L power:+5V #PWR0806
 U 1 1 5EEEAC0A
 P 5150 1550
-F 0 "#PWR?" H 5150 1400 50  0001 C CNN
+F 0 "#PWR0806" H 5150 1400 50  0001 C CNN
 F 1 "+5V" H 5165 1723 50  0000 C CNN
 F 2 "" H 5150 1550 50  0001 C CNN
@@
 $EndComp
 $Comp
-L power:VBUS #PWR?
+L power:VBUS #PWR0804
 U 1 1 5EEEB1B1
 P 4600 1550
-F 0 "#PWR?" H 4600 1400 50  0001 C CNN
+F 0 "#PWR0804" H 4600 1400 50  0001 C CNN
 F 1 "VBUS" H 4615 1723 50  0000 C CNN
 F 2 "" H 4600 1550 50  0001 C CNN
