File: Red/Red.sch (KiCad schematic (older format))
At the start: 5 parts

Commit message: Post design review
Parts:
- removed JP101: Jumper_2_Bridged, digikey-kicad-library:PinHeader_1x2_P2.54mm, symbol Jumper:Jumper_2_Bridged
Changed lines of the file:
@@
 Wire Wire Line
 	4750 3550 4100 3550
-Connection ~ 4650 3900
-Wire Wire Line
-	4650 3650 4650 3900
-Wire Wire Line
-	4100 3650 4650 3650
-$Sheet
-S 3600 2800 500  850
-U 5EC43DD6
-F0 "IOConnector" 50
-F1 "IOConnector.sch" 50
-F2 "USB_D-" I R 4100 2950 50
-F3 "USB_D+" I R 4100 2850 50
-F4 "SDA" I R 4100 3250 50
-F5 "SCL" I R 4100 3350 50
-F6 "USART_RX" I R 4100 3150 50
-F7 "USART_TX" I R 4100 3050 50
-F8 "D1" I R 4100 3450 50
-F9 "D2" I R 4100 3550 50
-F10 "D3" I R 4100 3650 50
-$EndSheet
-Wire Wire Line
-	4200 3900 4250 3900
-Wire Wire Line
-	4200 4150 4200 3900
-Wire Wire Line
-	4100 4150 4200 4150
-Wire Wire Line
-	4650 3900 4750 3900
-$Comp
-L Jumper:Jumper_2_Bridged JP101
-U 1 1 5EC38C4C
-P 4450 3900
-F 0 "JP101" H 4300 3800 50  0000 C CNN
-F 1 "Jumper_2_Bridged" H 4000 3950 50  0000 C CNN
-F 2 "digikey-kicad-library:PinHeader_1x2_P2.54mm" H 4450 3900 50  0001 C CNN
-F 3 "~" H 4450 3900 50  0001 C CNN
-F 4 "732-5315-ND" H 4450 3900 50  0001 C CNN "digikey"
-	1    4450 3900
-	1    0    0    -1
-$EndComp
 Wire Wire Line
 	4750 4650 4100 4650
@@
 	4100 4550 4750 4550
 Wire Wire Line
-	4750 4450 4100 4450
+	4750 4450 4550 4450
 Wire Wire Line
-	4100 4350 4750 4350
+	4100 4350 4600 4350
 Wire Wire Line
-	4750 4250 4100 4250
+	4750 4250 4650 4250
 $Sheet
 S 3600 4050 500  850
@@
 F0 "Sensors" 50
 F1 "Sensors.sch" 50
-F2 "INT1" I R 4100 4150 50
+F2 "INT1" I R 4100 4750 50
 F3 "~IMU_CS" I R 4100 4550 50
 F4 "SCLK" I R 4100 4250 50
@@
 F0 "Microprocessor" 50
 F1 "Microprocessor.sch" 50
-F2 "USB_D+" I L 4750 2850 50
-F3 "USB_D-" I L 4750 2950 50
+F2 "USART_RTS" I L 4750 2850 50
+F3 "USART_CTS" I L 4750 2950 50
 F4 "USART_RX" I L 4750 3150 50
 F5 "USART_TX" I L 4750 3050 50
@@
 F19 "MISO" I L 4750 4350 50
 F20 "MOSI" I L 4750 4450 50
-F21 "D3" I L 4750 3900 50
+F21 "INTERUPT" I L 4750 4750 50
 F22 "SDA" I L 4750 3250 50
 F23 "SCL" I L 4750 3350 50
@@
 F29 "QSPI_IO[0...3]" I R 6250 4850 50
 $EndSheet
+$Sheet
+S 3600 2550 500  1350
+U 5ED475E4
+F0 "IOConnector" 50
+F1 "IOConnector.sch" 50
+F2 "SDA" I R 4100 3250 50
+F3 "SCL" I R 4100 3350 50
+F4 "SCLK" I R 4100 3650 50
+F5 "MOSI" I R 4100 3850 50
+F6 "D1" I R 4100 3450 50
+F7 "D2" I R 4100 3550 50
+F8 "TXD" I R 4100 3150 50
+F9 "RXD" I R 4100 3050 50
+F10 "~RTS~" I R 4100 2950 50
+F11 "~CTS~" I R 4100 2850 50
+F12 "MISO" I R 4100 3750 50
+$EndSheet
+Wire Wire Line
+	4750 4750 4100 4750
+Wire Wire Line
+	4100 3650 4650 3650
+Wire Wire Line
+	4650 3650 4650 4250
+Connection ~ 4650 4250
+Wire Wire Line
+	4650 4250 4100 4250
+Wire Wire Line
+	4100 3750 4600 3750
+Wire Wire Line
+	4600 3750 4600 4350
+Connection ~ 4600 4350
+Wire Wire Line
+	4600 4350 4750 4350
+Wire Wire Line
+	4100 3850 4550 3850
+Wire Wire Line
+	4550 3850 4550 4450
+Connection ~ 4550 4450
+Wire Wire Line
+	4550 4450 4100 4450
 $EndSCHEMATC

Commit message: Created V1.1 Layout, minor schematic updates
Parts:
- removed H103, H104: MountingHole, MountingHole:MountingHole_4.3mm_M4, symbol Mechanical:MountingHole
Changed lines of the file:
@@
-	1    0    0    -1
-$EndComp
-$Comp
-L Mechanical:MountingHole H103
-U 1 1 5ED48920
-P 7750 5800
-F 0 "H103" H 7850 5846 50  0001 L CNN
-F 1 "MountingHole" H 7850 5755 50  0001 L CNN
-F 2 "MountingHole:MountingHole_4.3mm_M4" H 7750 5800 50  0001 C CNN
-F 3 "~" H 7750 5800 50  0001 C CNN
-	1    7750 5800
-	1    0    0    -1
-$EndComp
-$Comp
-L Mechanical:MountingHole H104
-U 1 1 5ED48A5D
-P 7750 6100
-F 0 "H104" H 7850 6146 50  0001 L CNN
-F 1 "MountingHole" H 7850 6055 50  0001 L CNN
-F 2 "MountingHole:MountingHole_4.3mm_M4" H 7750 6100 50  0001 C CNN
-F 3 "~" H 7750 6100 50  0001 C CNN
-	1    7750 6100
 	1    0    0    -1
 $EndComp
