File: Red/Red.kicad_pcb (KiCad board)
At the start: 4 copper layers, 44 x 67.5 mm, 82 parts, among them IC701 STM32G473CET6, J201 Conn_01x02, J301 Conn_01x03, J302 Screw_Terminal_01x02, J303 Screw_Terminal_01x02, J701 Conn_01x06, J801 USB_C_Receptacle, J802 Conn_01x10, J803 Conn_01x10, Q301 DMG3414U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

Commit message: minor fixes
Routing:
- net /IOConnector/USBD-: track 10.2 -> 12.9 mm, vias 0 -> 1
- net /IOConnector/USBD+: track 8.11 -> 10.1 mm, vias 0 -> 1
- net /IOConnector/MISO: track 46.6 -> 45.9 mm
